File: 7segment_MultiMater_v3.kicad_sch (KiCad schematic)
At the start: 86 parts, among them J1 Conn_01x04_Socket, J2 GearPosition, P1 USB_C_Plug_USB2.0, Q1 IRLML6402, U1 SA10-21SRWA, U2 W25Q16JVUXIQ, U3 TB62706BF, U4 74HC595, U5 NJM12877F33, U6 MCP25625x-x-SS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

Commit message: 微修正
Changed lines of the file:
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@@
-	)
-	(junction
-		(at 229.87 132.08)
-		(diameter 0)
-		(color 0 0 0 0)
 	)
 	(junction
@@
 	(wire
 		(pts
-			(xy 229.87 123.19) (xy 229.87 132.08)
-		)
-		(stroke
-			(width 0)
-			(type default)
-		)
-	)
-	(wire
-		(pts
 			(xy 365.76 25.4) (xy 365.76 27.94)
 		)
@@
 	(wire
 		(pts
-			(xy 229.87 132.08) (xy 229.87 133.35)
+			(xy 229.87 123.19) (xy 229.87 133.35)
 		)
 		(stroke
@@
 		)
 		(stroke
-			(width 0)
-			(type default)
-		)
-	)
-	(wire
-		(pts
-			(xy 226.06 132.08) (xy 229.87 132.08)
-		)
-		(stroke
